File: aif_rc_teleop_ecu.kicad_sch (KiCad schematic)
At the start: 0 parts

Commit message: wip: 回路図作成作業中
Parts:
- added C1: 10μ, Package_QFP:PQFP-160_28x28mm_P0.65mm, symbol Device:C
- added C2: 0.1μ, symbol Device:C
- added J1: B02B-XASK-1, symbol Connector_Generic:Conn_01x02
- added J2: Conn_01x04, symbol Connector_Generic:Conn_01x04
Connections:
- new net +5V: C1.1, C2.2, J1.2 (Pin_2), J2.2 (Pin_2)
- new net GND: C1.2, C2.1, J1.1 (Pin_1), J2.1 (Pin_1)
- new net USART_RX: J2.4 (Pin_4)
- new net USART_TX: J2.3 (Pin_3)

Commit message: wip: 作業中
Parts:
- added J3: ST-LINK, symbol Connector_Generic:Conn_02x07_Odd_Even
- J1: value B02B-XASK-1 -> PWR
Connections:
- net GND: now also J3.5 (Pin_5), J3.7 (Pin_7)
- new net +3.3V: J3.3 (Pin_3)
- new net SWCLK: J3.6 (Pin_6)
- new net SWDIO: J3.4 (Pin_4)
- new net SWO: J3.8 (Pin_8)
- no-connect marks 0 -> 8
Other:
- added sheet STM32G474 (STM32G474.kicad_sch)

Commit message: wip: 回路図作成作業中
Parts:
- added J4: CAN, symbol Connector_Generic:Conn_01x03
- added JP1: Jumper_2_Open, Package_LCC:PLCC-84_29.3x29.3mm_P1.27mm, symbol Jumper:Jumper_2_Open
- added R1: 120, symbol Device:R
Connections:
- net USART_RX: now also J2.3 (Pin_3); no longer J2.4 (Pin_4)
- net USART_TX: now also J2.4 (Pin_4); no longer J2.3 (Pin_3)
- net SWCLK renamed STM32G474/SWCLK
- net SWDIO renamed STM32G474/SWDIO
- net SWO renamed STM32G474/SWO
- new net: JP1.1 (A), R1.1
- new net CAN_Transeiver/CAN_H: J4.2 (Pin_2), JP1.2 (B)
- new net CAN_Transeiver/CAN_L: J4.3 (Pin_3), R1.2
- new net CAN_Transeiver/GND_CAN: J4.1 (Pin_1)
Other:
- added sheet CAN_Transeiver (ISOW1044.kicad_sch)
- added sheet PWR (PWR.kicad_sch)
- sheet STM32G474 ports: added CAN_RX, CAN_TX, NRST, SWCLK, SWDIO, SWO, USART_RX, USART_TX; removed none

Commit message: feat: 回路図一旦完成
Parts:
- added SW1: SW_Push, Button_Switch_SMD:SW_Push_1P1T_XKB_TS-1187A, symbol Switch:SW_Push
- C1: footprint Package_QFP:PQFP-160_28x28mm_P0.65mm -> Capacitor_SMD:C_0805_2012Metric
- C2: footprint (none) -> Capacitor_SMD:C_0603_1608Metric
- J1: footprint (none) -> Connector_JST:JST_XA_B02B-XASK-1_1x02_P2.50mm_Vertical
- J2: footprint (none) -> Connector_PinHeader_2.54mm:PinHeader_1x04_P2.54mm_Vertical
- J3: footprint (none) -> Connector_PinHeader_1.27mm:PinHeader_2x07_P1.27mm_Vertical_SMD
- J4: footprint (none) -> Connector_JST:JST_XA_B03B-XASK-1_1x03_P2.50mm_Vertical
- JP1: footprint Package_LCC:PLCC-84_29.3x29.3mm_P1.27mm -> Connector_PinHeader_2.54mm:PinHeader_1x02_P2.54mm_Vertical
- R1: footprint (none) -> Resistor_SMD:R_0603_1608Metric
Connections:
- net GND: now also SW1.1
- net STM32G474/NRST: now also J3.12 (Pin_12), SW1.2
- net USART_RX: now also J2.4 (Pin_4); no longer J2.3 (Pin_3)
- net USART_TX: now also J2.3 (Pin_3); no longer J2.4 (Pin_4)
- no-connect marks 8 -> 7
Other:
- moved on the sheet: J3

Commit message: wip: pcb作業中
Parts:
- added H1, H2, H3, H4: MountingHole, MountingHole:MountingHole_3.2mm_M3, symbol Mechanical:MountingHole

Commit message: wip: 作業中
Parts:
- J3: footprint Connector_PinHeader_1.27mm:PinHeader_2x07_P1.27mm_Vertical_SMD -> my_pretty:JTAG_BOX_CONN
Changed lines of the file:
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@@
 			)
 		)
-		(property "Footprint" "Connector_PinHeader_1.27mm:PinHeader_2x07_P1.27mm_Vertical_SMD"
+		(property "Footprint" "my_pretty:JTAG_BOX_CONN"
 			(at 38.1 109.22 0)
 			(hide yes)

Commit message: fix: バグ修正
Connections:
- net CAN_Transeiver/CAN_H renamed CA-IS3062VW/CAN_H
- net CAN_Transeiver/CAN_L renamed CA-IS3062VW/CAN_L
- net CAN_Transeiver/GND_CAN renamed CA-IS3062VW/GND_CAN
Other:
- removed sheet CAN_Transeiver
- added sheet CA-IS3062VW (CA-IS3062VW.kicad_sch)
Changed lines of the file:
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@@
 			(color 0 0 0 0)
 		)
-		(property "Sheetname" "CAN_Transeiver"
+		(property "Sheetname" "CA-IS3062VW"
 			(at 60.96 146.6084 0)
 			(show_name no)
@@
 			)
 		)
-		(property "Sheetfile" "ISOW1044.kicad_sch"
+		(property "Sheetfile" "CA-IS3062VW.kicad_sch"
 			(at 60.96 177.1146 0)
 			(show_name no)

Commit message: feat: 回路図pdf追加
Other:
- sheet CA-IS3062VW renamed CAN_Transeiver
Changed lines of the file:
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@@
 			(color 0 0 0 0)
 		)
-		(property "Sheetname" "CA-IS3062VW"
+		(property "Sheetname" "CAN_Transeiver"
 			(at 60.96 146.6084 0)
 			(show_name no)
