File: aif_rc_teleop_ecu.kicad_sch (KiCad schematic)
At the start: 13 parts, among them J1 PWR, J2 Conn_01x04, J3 ST-LINK, J4 CAN, SW1 SW_Push

Commit message: feat: pcb再設計
Parts:
- J2: footprint Connector_PinHeader_2.54mm:PinHeader_1x04_P2.54mm_Vertical -> Connector_JST:JST_XA_B04B-XASK-1_1x04_P2.50mm_Vertical
Changed lines of the file:
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@@
 			)
 		)
-		(property "Footprint" "Connector_PinHeader_2.54mm:PinHeader_1x04_P2.54mm_Vertical"
+		(property "Footprint" "Connector_JST:JST_XA_B04B-XASK-1_1x04_P2.50mm_Vertical"
 			(at 195.58 68.58 0)
 			(hide yes)
