File: CA-IS3062VW.kicad_sch (KiCad schematic)
At the start: 8 parts, among them U3 CA-IS3062VW

Commit message: feat: 回路図pdf追加
Other:
- note removed: "CA-IS3062VW 絶縁CANトランシーバ（データシート Ver.1.08） ・VCC=+5V（4.5〜5.5V, p.5）、VCCL=+3.3V（2.375〜5.5V, p.5 / VCCとは別電圧可 p.4 注1） ・TXD VIH=2V（p.5）→ 3.3V MCUと直結可 ・VCC, VISO(16) は 0.1µF||10µF（p.20）。10µFはピンから2mm以内、ICと同一面・ビア無し（p.20） ・VCCL は 1µF X5R/X7R（p.20） ・VISO(16)→ビーズ→VISO(11)、11番に 1µF を最短で配置（p.19 図10-1, p.20 図10-3） ・NC(4,6,14) は未接続（p.4） ・終端抵抗はメインシートの R1/JP1（p.19 単一120Ω終端）"
- moved on the sheet: C19, C20

Commit message: feat: pcb再設計
Parts:
- C19, C22: value 10u -> 10μ
- C20, C23: value 0.1u -> 0.1μ
- C21, C24: value 1u -> 1μ
Changed lines of the file:
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@@
 			)
 		)
-		(property "Value" "10u"
+		(property "Value" "10μ"
 			(at 203.2 96.52 0)
 			(show_name no)
@@
 			)
 		)
-		(property "Value" "1u"
+		(property "Value" "1μ"
 			(at 123.19 121.92 0)
 			(show_name no)
@@
 			)
 		)
-		(property "Value" "1u"
+		(property "Value" "1μ"
 			(at 175.26 109.22 0)
 			(show_name no)
@@
 			)
 		)
-		(property "Value" "0.1u"
+		(property "Value" "0.1μ"
 			(at 210.82 96.52 0)
 			(show_name no)
@@
 			)
 		)
-		(property "Value" "0.1u"
+		(property "Value" "0.1μ"
 			(at 128.27 86.36 0)
 			(show_name no)
@@
 			)
 		)
-		(property "Value" "10u"
+		(property "Value" "10μ"
 			(at 119.38 86.36 0)
 			(show_name no)
