File: PWR.kicad_sch (KiCad schematic)
At the start: 8 parts, among them U2 XC6206PxxxMR

Commit message: feat: 回路図一旦完成
Parts:
- C3: footprint (none) -> Capacitor_THT:CP_Radial_D6.3mm_P2.50mm
- C4: footprint Package_TO_SOT_SMD:SOT-23-3 -> Capacitor_SMD:C_0603_1608Metric
- C5: footprint (none) -> Capacitor_SMD:C_0603_1608Metric
- D3: footprint LED_SMD:LED_Cree-XHP50_3V_HighDensity -> LED_SMD:LED_0805_2012Metric
- D4: footprint (none) -> LED_SMD:LED_0805_2012Metric
- R2, R3: footprint (none) -> Resistor_SMD:R_0603_1608Metric
- U2: value XC6206PxxxMR -> XC6206P332MR
Changed lines of the file:
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@@
 			)
 		)
-		(property "Footprint" ""
+		(property "Footprint" "Resistor_SMD:R_0603_1608Metric"
 			(at 174.752 99.06 90)
 			(hide yes)
@@
 			)
 		)
-		(property "Footprint" ""
+		(property "Footprint" "Resistor_SMD:R_0603_1608Metric"
 			(at 211.582 99.06 90)
 			(hide yes)
@@
 			)
 		)
-		(property "Footprint" ""
+		(property "Footprint" "Capacitor_THT:CP_Radial_D6.3mm_P2.50mm"
 			(at 40.3352 119.38 0)
 			(hide yes)
@@
 			)
 		)
-		(property "Footprint" ""
+		(property "Footprint" "Capacitor_SMD:C_0603_1608Metric"
 			(at 103.8352 119.38 0)
 			(hide yes)
@@
 			)
 		)
-		(property "Footprint" "Package_TO_SOT_SMD:SOT-23-3"
+		(property "Footprint" "Capacitor_SMD:C_0603_1608Metric"
 			(at 60.6552 119.38 0)
 			(hide yes)
@@
 			)
 		)
-		(property "Footprint" ""
+		(property "Footprint" "LED_SMD:LED_0805_2012Metric"
 			(at 213.36 110.49 0)
 			(hide yes)
@@
 			)
 		)
-		(property "Footprint" "LED_SMD:LED_Cree-XHP50_3V_HighDensity"
+		(property "Footprint" "LED_SMD:LED_0805_2012Metric"
 			(at 176.53 110.49 0)
 			(hide yes)
@@
 			)
 		)
-		(property "Value" "XC6206PxxxMR"
+		(property "Value" "XC6206P332MR"
 			(at 81.28 97.79 0)
 			(show_name no)

Commit message: feat: pcb再設計
Parts:
- C3: value 100u -> 100μ
- C4, C5: value 1u -> 1μ
- D3, D4: footprint LED_SMD:LED_0805_2012Metric -> LED_SMD:LED_0603_1608Metric
Changed lines of the file:
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@@
 			)
 		)
-		(property "Value" "100u"
+		(property "Value" "100μ"
 			(at 43.18 116.8399 0)
 			(show_name no)
@@
 			)
 		)
-		(property "Value" "1u"
+		(property "Value" "1μ"
 			(at 106.68 116.8399 0)
 			(show_name no)
@@
 			)
 		)
-		(property "Value" "1u"
+		(property "Value" "1μ"
 			(at 63.5 116.8399 0)
 			(show_name no)
@@
 			)
 		)
-		(property "Footprint" "LED_SMD:LED_0805_2012Metric"
+		(property "Footprint" "LED_SMD:LED_0603_1608Metric"
 			(at 213.36 110.49 0)
 			(hide yes)
@@
 			)
 		)
-		(property "Footprint" "LED_SMD:LED_0805_2012Metric"
+		(property "Footprint" "LED_SMD:LED_0603_1608Metric"
 			(at 176.53 110.49 0)
 			(hide yes)
