File: STM32G474.kicad_sch (KiCad schematic)
At the start: 0 parts

Commit message: wip: 回路図作成作業中
Parts:
- added C6: 0.1μ, symbol Device:C
- added U1: STM32G474RETx, Package_QFP:LQFP-64_10x10mm_P0.5mm, symbol MCU_ST_STM32G4:STM32G474RETx
Connections:
- new net: U1.15 (VSS), U1.31 (VSS), U1.47 (VSS), U1.63 (VSS)
- new net CAN_RX: U1.45 (PA11)
- new net CAN_TX: U1.46 (PA12)
- new net GND: C6.2
- new net NRST: C6.1, U1.7 (PG10)
- new net USART_RX: U1.60 (PB7)
- new net USART_TX: U1.59 (PB6)

Commit message: feat: 回路図一旦完成
Parts:
- added C10, C11, C12, C14, C9: 100n, Capacitor_SMD:C_0603_1608Metric, symbol Device:C
- added C13: 4.7μ, Capacitor_SMD:C_0603_1608Metric, symbol Device:C
- added C15, C8: 1μ, Capacitor_SMD:C_0603_1608Metric, symbol Device:C
- added C7: 10n, Capacitor_SMD:C_0603_1608Metric, symbol Device:C
- added D1, D2, D5: LED, LED_SMD:LED_0805_2012Metric, symbol Device:LED
- added L1: 600@100MHz, Resistor_SMD:R_0805_2012Metric, symbol Device:L_Ferrite
- added R4, R5, R6: 1.2k, Resistor_SMD:R_0603_1608Metric, symbol Device:R
- added R7: 10k, Resistor_SMD:R_0603_1608Metric, symbol Device:R
- C6: footprint (none) -> Capacitor_SMD:C_0603_1608Metric
Connections:
- net GND: now also U1.15 (VSS), U1.27 (VSSA), U1.31 (VSS), U1.47 (VSS), U1.63 (VSS), C10.2, C11.2, C12.2, C13.2, C14.2, C15.2, C7.2, C8.2, C9.2, D1.1 (K), D2.1 (K), D5.1 (K), R7.2
- net SWCLK: now also U1.50 (PA14)
- net SWDIO: now also U1.49 (PA13)
- net SWO: now also U1.56 (PB3)
- net +3.3V: now reaches U1.1 (VBAT)
- net +3.3V: now also U1.16 (VDD), U1.32 (VDD), U1.48 (VDD), U1.64 (VDD), C10.1, C11.1, C12.1, C13.1, C9.1, L1.1
- net STATUS_LED: now reaches U1.24 (PB0)
- net STATUS_LED: now also R4.1
- net FAIL_LED: now reaches U1.25 (PB1)
- net FAIL_LED: now also R5.1
- net MODE_LED: now reaches U1.26 (PB2)
- net MODE_LED: now also R6.1
- net VDDA: now reaches U1.28 (VREF+)
- net VDDA: now also U1.29 (VDDA), C14.1, C15.1, C7.1, C8.1, L1.2
- net at U1.61 (PB8): now also R7.1
- new net: D1.2 (A), R4.2
- new net: D2.2 (A), R5.2
- new net: D5.2 (A), R6.2
- no-connect marks 0 -> 40

Commit message: feat: 水晶振動子追加とer6ピンをxaコネクタに変更
Parts:
- removed L1: 600@100MHz, Resistor_SMD:R_0805_2012Metric, symbol Device:L_Ferrite
- added C16, C17: 20p, Capacitor_SMD:C_0603_1608Metric, symbol Device:C
- added R8: 0, Resistor_SMD:R_0603_1608Metric, symbol Device:R
- added Y1: 8MHz, Crystal:Crystal_SMD_5032-2Pin_5.0x3.2mm, symbol Device:Crystal
Connections:
- net VDDA is gone; now on net +3.3V: C14.1, C15.1, C7.1, C8.1, U1.28 (VREF+), U1.29 (VDDA)
- net GND: now also C16.1, C17.1
- net at U1.5 (PF0): now also C16.2, Y1.2
- net at U1.6 (PF1): now also R8.2
- new net: C17.2, R8.1, Y1.1
- no-connect marks 40 -> 38
Other:
- moved on the sheet: C6

Commit message: feat: pcb再設計
Parts:
- removed R8: 0, Resistor_SMD:R_0603_1608Metric, symbol Device:R
- C10, C11, C12, C14, C9: value 100n -> 0.1μ
- C16, C17: value 20p -> 33p
- D1, D2, D5: footprint LED_SMD:LED_0805_2012Metric -> LED_SMD:LED_0603_1608Metric
Connections:
- net at C17.2, Y1.1: now also U1.6 (PF1)
Changed lines of the file:
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@@
 	(wire
 		(pts
-			(xy 92.71 74.93) (xy 93.98 74.93)
-		)
-		(stroke
-			(width 0)
-			(type default)
-		)
-	)
-	(wire
-		(pts
 			(xy 215.9 102.87) (xy 215.9 106.68)
 		)
@@
 	(wire
 		(pts
-			(xy 80.01 74.93) (xy 85.09 74.93)
+			(xy 80.01 74.93) (xy 93.98 74.93)
 		)
 		(stroke
@@
 			)
 		)
-		(property "Value" "100n"
+		(property "Value" "0.1μ"
 			(at 222.25 44.4499 0)
 			(show_name no)
@@
 			)
 		)
-		(property "Value" "100n"
+		(property "Value" "0.1μ"
 			(at 71.12 40.6399 0)
 			(show_name no)
@@
 			)
 		)
-		(property "Value" "100n"
+		(property "Value" "0.1μ"
 			(at 210.82 44.4499 0)
 			(show_name no)
@@
 			)
 		)
-		(property "Footprint" "LED_SMD:LED_0805_2012Metric"
+		(property "Footprint" "LED_SMD:LED_0603_1608Metric"
 			(at 184.15 110.49 0)
 			(hide yes)
@@
 			)
 		)
-		(property "Footprint" "LED_SMD:LED_0805_2012Metric"
+		(property "Footprint" "LED_SMD:LED_0603_1608Metric"
 			(at 199.39 110.49 0)
 			(hide yes)
@@
 	)
 	(symbol
-		(lib_id "Device:R")
-		(at 88.9 74.93 90)
-		(unit 1)
-		(body_style 1)
-		(exclude_from_sim no)
-		(in_bom yes)
-		(on_board yes)
-		(in_pos_files yes)
-		(dnp no)
-		(property "Reference" "R8"
-			(at 92.202 77.47 90)
-			(show_name no)
-			(do_not_autoplace no)
-			(effects
-				(font
-					(size 1.27 1.27)
-				)
-			)
-		)
-		(property "Value" "0"
-			(at 88.9 77.978 90)
-			(show_name no)
-			(do_not_autoplace no)
-			(effects
-				(font
-					(size 1.27 1.27)
-				)
-			)
-		)
-		(property "Footprint" "Resistor_SMD:R_0603_1608Metric"
-			(at 88.9 76.708 90)
-			(hide yes)
-			(show_name no)
-			(do_not_autoplace no)
-			(effects
-				(font
-					(size 1.27 1.27)
-				)
-			)
-		)
-		(property "Datasheet" ""
-			(at 88.9 74.93 0)
-			(hide yes)
-			(show_name no)
-			(do_not_autoplace no)
-			(effects
-				(font
-					(size 1.27 1.27)
-				)
-			)
-		)
-		(property "Description" "Resistor"
-			(at 88.9 74.93 0)
-			(hide yes)
-			(show_name no)
-			(do_not_autoplace no)
-			(effects
-				(font
-					(size 1.27 1.27)
-				)
-			)
-		)
-		(pin "2"
-		)
-		(pin "1"
-		)
-		(instances
-			(project "aif_rc_teleop_ecu"
-				(path "/a363d9db-65ec-4e34-8378-615a57ba2446/0cdf92b2-bee3-4bd4-9ef9-48bd503d20b2"
-					(reference "R8")
-					(unit 1)
-				)
-			)
-		)
-	)
-	(symbol
 		(lib_id "power:+3.3V")
 		(at 67.31 29.21 0)
@@
 			)
 		)
-		(property "Value" "100n"
+		(property "Value" "0.1μ"
 			(at 187.96 44.4499 0)
 			(show_name no)
@@
 			)
 		)
-		(property "Value" "20p"
+		(property "Value" "33p"
 			(at 65.532 61.468 90)
 			(show_name no)
@@
 			)
 		)
-		(property "Footprint" "LED_SMD:LED_0805_2012Metric"
+		(property "Footprint" "LED_SMD:LED_0603_1608Metric"
 			(at 215.9 110.49 0)
 			(hide yes)
@@
 			)
 		)
-		(property "Value" "100n"
+		(property "Value" "0.1μ"
 			(at 199.39 44.4499 0)
 			(show_name no)
@@
 			)
 		)
-		(property "Value" "20p"
+		(property "Value" "33p"
 			(at 68.834 78.74 90)
 			(show_name no)

Commit message: fix: 添削内容を踏まえて修正
Connections:
- net FAIL_LED: now also U1.18 (PA4); no longer U1.25 (PB1)
- net MODE_LED: now also U1.19 (PA5); no longer U1.26 (PB2)
- net STATUS_LED: now also U1.17 (PA3); no longer U1.24 (PB0)
Changed lines of the file:
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@@
 	)
 	(no_connect
-		(at 135.89 62.23)
+		(at 135.89 97.79)
 	)
 	(no_connect
@@
 	)
 	(no_connect
-		(at 135.89 59.69)
+		(at 135.89 95.25)
 	)
 	(no_connect
@@
 	)
 	(no_connect
-		(at 135.89 57.15)
+		(at 135.89 92.71)
 	)
 	(no_connect
@@
 	(wire
 		(pts
-			(xy 135.89 97.79) (xy 139.7 97.79)
+			(xy 135.89 62.23) (xy 139.7 62.23)
 		)
 		(stroke
@@
 	(wire
 		(pts
-			(xy 135.89 95.25) (xy 139.7 95.25)
+			(xy 135.89 59.69) (xy 139.7 59.69)
 		)
 		(stroke
@@
 	(wire
 		(pts
-			(xy 135.89 92.71) (xy 139.7 92.71)
+			(xy 135.89 57.15) (xy 139.7 57.15)
 		)
 		(stroke
@@
 	)
 	(label "MODE_LED"
-		(at 139.7 97.79 0)
+		(at 139.7 62.23 0)
 		(effects
 			(font
@@
 	)
 	(label "FAIL_LED"
-		(at 139.7 95.25 0)
+		(at 139.7 59.69 0)
 		(effects
 			(font
@@
 	)
 	(label "STATUS_LED"
-		(at 139.7 92.71 0)
+		(at 139.7 57.15 0)
 		(effects
 			(font
