File: aif_rc_teleop_ecu.kicad_pcb (KiCad board)
At the start: 2 copper layers, 80 x 55.5 mm, 57 parts, among them IC1 ISOW1044BDFMR, J1 PWR, J2 Conn_01x04, J3 ST-LINK, J4 CAN, SW1 SW_Push, U1 STM32G474RETx, U2 XC6206P332MR

Commit message: wip: 作業中
Parts:
- J3: footprint Connector_PinHeader_1.27mm:PinHeader_2x07_P1.27mm_Vertical_SMD -> my_pretty:JTAG_BOX_CONN
- moved SW1 35.6 mm to (158.2, 79.3), turned to 180 degrees
- moved J3 13.0 mm to (196.9, 75.0), turned to 90 degrees
- moved D1 1.80 mm to (155.9, 60.2)
- moved R4 1.80 mm to (160.9, 60.2)
- moved L1 1.58 mm to (156.9, 75.2)
- moved C10 1.53 mm to (162.4, 73.0), turned to -90 degrees
- moved C7 1.49 mm to (162.4, 69.8), turned to 90 degrees
- moved C8 1.35 mm to (160.0, 72.4)
- moved C11 1.04 mm to (174.5, 75.6), turned to 0 degrees
- moved C15 1.03 mm to (156.9, 72.4)
- moved D3 1.00 mm to (184.6, 55.6)
- moved D4 1.00 mm to (188.8, 55.6)
- moved D2 0.60 mm to (155.9, 63.4)
- moved R5 0.60 mm to (160.9, 63.4)
- moved D5 0.60 mm to (155.9, 66.6)
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Routing:
- net +5V: track 0.00 -> 102.0 mm, vias 0 -> 3
- net +3.3V: track 0.00 -> 98.6 mm
- net /STM32G474/NRST: track 0.00 -> 51.1 mm, vias 0 -> 2
- net GND: track 0.00 -> 33.9 mm, vias 0 -> 195
- net /CAN_Transeiver/CAN_L: track 0.00 -> 25.9 mm
- net /USART_RX: track 0.00 -> 20.7 mm
- net Net-(IC1-VISOIN): track 0.00 -> 20.6 mm, vias 0 -> 2
- net /USART_TX: track 0.00 -> 19.9 mm
- net /CAN_Transeiver/CAN_H: track 0.00 -> 17.5 mm
- net VDDA: track 0.00 -> 16.2 mm
- net /STM32G474/SWO: track 0.00 -> 14.9 mm
- net Net-(IC1-VDD): track 0.00 -> 14.1 mm, vias 0 -> 2
- net Net-(IC1-GND1): track 0.00 -> 13.9 mm
- net Net-(IC1-VISOOUT): track 0.00 -> 13.2 mm
- net Net-(IC1-GND2): track 0.00 -> 12.4 mm
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Other:
- board text added: "3.3V"
- board text added: "5V"
- board text added: "AIF_RC遠隔操縦基板 Ver.0.0 設計：kyo0221"
- board text added: "CAN"
- board text added: "ER6"
- board text added: "ST-LINK"
- board text added: "モード"
- board text added: "状態"
- board text added: "異常"
- board text added: "終端抵抗"
- board text added: "電源表示"
- board text removed: "AIF_RC遠隔操縦基板 v0.0 設計者：kyo0221"
- board text removed: "ANT ->"
- board text removed: "CAN ISO"
- board text removed: "ER6 AREA"

Commit message: feat: 回路図pdf追加
Parts:
- removed C25, C27: 10u, Capacitor_SMD:C_0603_1608Metric
- removed C26: 1u, Capacitor_SMD:C_0603_1608Metric
- removed FB2, FB3, FB4, FB5: FerriteBead, Inductor_SMD:L_0402_1005Metric
- removed IC1: ISOW1044BDFMR, Package_SO:SOIC-20W_7.5x12.8mm_P1.27mm
- removed R14: 4.7k, Resistor_SMD:R_0603_1608Metric
- added U3: CA-IS3062VW, Package_SO:SOIC-16W_7.5x10.3mm_P1.27mm, F.Cu at (175.0, 88.0)
- C19: footprint Capacitor_SMD:C_0603_1608Metric -> Capacitor_SMD:C_0805_2012Metric
- C20: value 1u -> 0.1u
- C21, C24: value 10n -> 1u
- C22: value 0.1u -> 10u; footprint Capacitor_SMD:C_0603_1608Metric -> Capacitor_SMD:C_0805_2012Metric
- FB1: value FerriteBead -> 330@100MHz
- moved H4 31.5 mm to (194.5, 99.3)
- moved H2 31.5 mm to (194.5, 54.3)
- moved FB1 17.1 mm to (171.2, 95.9), turned to 0 degrees
- moved C19 16.7 mm to (182.3, 83.3), turned to 0 degrees
- moved C22 12.3 mm to (182.3, 92.6), turned to 0 degrees
- moved C20 11.1 mm to (178.8, 81.2), turned to 180 degrees
- moved G*** 4.00 mm to (159.5, 87.0)
- moved C24 2.41 mm to (173.1, 95.6), turned to -90 degrees
- moved JP1 1.72 mm to (187.9, 98.4)
- moved J4 1.72 mm to (182.5, 99.2)
- moved H3 1.70 mm to (155.0, 99.3)
- moved C21 1.57 mm to (170.3, 81.0), turned to 180 degrees
- moved C23 1.39 mm to (182.1, 94.5), turned to 0 degrees
- moved R1 0.95 mm to (187.9, 94.0)
Connections:
- C19 pad 1: Net-(IC1-VDD) -> +5V
- C19 pad 2: Net-(IC1-GND1) -> GND
- C20 pad 1: Net-(IC1-VDD) -> +5V
- C20 pad 2: Net-(IC1-GND1) -> GND
- C21 pad 1: Net-(IC1-VDD) -> +3.3V
- C21 pad 2: Net-(IC1-GND1) -> GND
- C22 pad 1: Net-(IC1-VIO) -> Net-(C22-Pad1)
- C22 pad 2: GND -> /CAN_Transeiver/GND_CAN
- C23 pad 1: Net-(IC1-VISOIN) -> Net-(C22-Pad1)
- C24 pad 1: Net-(IC1-VISOOUT) -> Net-(C24-Pad1)
- C24 pad 2: Net-(IC1-GND2) -> /CAN_Transeiver/GND_CAN
- FB1 pad 1: GND -> Net-(C22-Pad1)
- FB1 pad 2: Net-(IC1-GND1) -> Net-(C24-Pad1)
Routing:
- net Net-(IC1-VISOIN): track 20.6 -> 0.00 mm, vias 2 -> 0
- net Net-(C22-Pad1): track 0.00 -> 18.1 mm, vias 0 -> 2
- net +5V: track 102.0 -> 84.6 mm, vias 3 -> 1
- net +3.3V: track 98.6 -> 113.3 mm
- net Net-(IC1-VDD): track 14.1 -> 0.00 mm, vias 2 -> 0
- net Net-(IC1-GND1): track 13.9 -> 0.00 mm
- net Net-(IC1-VISOOUT): track 13.2 -> 0.00 mm
- net Net-(IC1-GND2): track 12.4 -> 0.00 mm
- net Net-(IC1-EN/FLT): track 5.32 -> 0.00 mm
- net Net-(IC1-VIO): track 4.94 -> 0.00 mm
- net Net-(C24-Pad1): track 0.00 -> 4.03 mm
- net /CAN_Transeiver/GND_CAN: track 5.40 -> 8.62 mm, vias 35 -> 13
- net GND: track 33.9 -> 36.3 mm, vias 195 -> 152
- net Net-(JP1-A): track 5.44 -> 3.62 mm
- net /CAN_Transeiver/CAN_TX: track 11.9 -> 11.4 mm
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Other:
- board size 80 x 55.5 mm -> 73.5 x 53 mm

Commit message: feat: 水晶振動子追加とer6ピンをxaコネクタに変更
Parts:
- added C16: 20p, Capacitor_SMD:C_0603_1608Metric, F.Cu at (1.50, 0.76)
- added C17: 20p, Capacitor_SMD:C_0603_1608Metric, F.Cu at (1.50, 3.27)
- added R8: 0, Resistor_SMD:R_0603_1608Metric, F.Cu at (1.50, 5.78)
- added Y1: 8MHz, Crystal:Crystal_SMD_5032-2Pin_5.0x3.2mm, F.Cu at (7.18, 2.12)
- J2: footprint Connector_PinHeader_2.54mm:PinHeader_1x04_P2.54mm_Vertical -> Connector_JST:JST_XA_B04B-XASK-1_1x04_P2.50mm_Vertical
Connections:
- C14 pad 1: VDDA -> +3.3V
- C15 pad 1: VDDA -> +3.3V
- C7 pad 1: VDDA -> +3.3V
- C8 pad 1: VDDA -> +3.3V
- U1 pad 28: VDDA -> +3.3V
- U1 pad 29: VDDA -> +3.3V
- U1 pad 5: unconnected-(U1-PF0-Pad5) -> Net-(U1-PF0)
- U1 pad 6: unconnected-(U1-PF1-Pad6) -> Net-(U1-PF1)
Routing:
- net GND: vias 152 -> 151
- net /USART_TX: vias 0 -> 1

Commit message: feat: pcb再設計
Parts:
- removed L1: 600@100MHz, Resistor_SMD:R_0805_2012Metric
- removed R8: 0, Resistor_SMD:R_0603_1608Metric
- C10, C11, C12, C14, C9: value 100n -> 0.1μ
- C16, C17: value 20p -> 33p
- C19, C22: value 10u -> 10μ
- C20, C23: value 0.1u -> 0.1μ
- C21, C24, C4, C5: value 1u -> 1μ
- C3: value 100u -> 100μ
- D1, D2, D3, D4, D5: footprint LED_SMD:LED_0805_2012Metric -> LED_SMD:LED_0603_1608Metric
- moved C16 187.2 mm to (175.0, 71.0), turned to -90 degrees
- moved C17 178.8 mm to (167.0, 71.0), turned to -90 degrees
- moved Y1 177.5 mm to (171.0, 70.4)
- moved FB1 40.8 mm to (195.6, 63.2), turned to -90 degrees
- moved D4 36.7 mm to (153.9, 67.0)
- moved C24 36.6 mm to (196.4, 67.3), turned to 0 degrees
- moved C22 36.6 mm to (196.6, 58.9)
- moved C23 36.4 mm to (196.4, 61.0)
- moved R3 34.8 mm to (157.4, 67.0), turned to 180 degrees
- moved D3 31.4 mm to (153.9, 62.2)
- moved C6 30.9 mm to (184.4, 87.4), turned to 90 degrees
- moved R2 29.1 mm to (157.4, 62.2), turned to 180 degrees
- moved U3 26.5 mm to (188.8, 65.4), turned to 0 degrees
- moved J4 25.3 mm to (195.0, 77.2)
- moved J2 24.3 mm to (173.0, 55.0), turned to 0 degrees
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Connections:
- C17 pad 2: Net-(C17-Pad2) -> Net-(U1-PF1)
- Y1 pad 1: Net-(C17-Pad2) -> Net-(U1-PF1)
Routing:
- net +5V: track 84.6 -> 0.00 mm, vias 1 -> 0
- net /CAN_Transeiver/CAN_RX: track 10.6 -> 60.1 mm
- net /CAN_Transeiver/CAN_TX: track 11.4 -> 51.2 mm
- net +3.3V: track 113.3 -> 137.2 mm, vias 0 -> 6
- net GND: track 36.3 -> 18.4 mm, vias 151 -> 76
- net VDDA: track 16.2 -> 0.00 mm
- net Net-(C22-Pad1): track 18.1 -> 5.94 mm, vias 2 -> 0
- net /CAN_Transeiver/CAN_L: track 25.4 -> 13.8 mm
- net /STM32G474/NRST: track 51.1 -> 40.5 mm, vias 2 -> 4
- net /USART_TX: track 19.9 -> 29.4 mm, vias 1 -> 6
- net Net-(JP1-A): track 3.62 -> 12.2 mm
- net /USART_RX: track 20.7 -> 28.2 mm, vias 0 -> 6
- net /CAN_Transeiver/GND_CAN: track 8.62 -> 15.5 mm, vias 13 -> 2
- net Net-(U1-PF1): track 0.00 -> 6.86 mm
- net Net-(U1-PF0): track 0.00 -> 6.81 mm
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- added copper zone on F.Cu, net +3.3V
- added copper zone on F.Cu, net +5V
- removed copper zone on B.Cu, net /CAN_Transeiver/GND_CAN
Other:
- board size 73.5 x 53 mm -> 48.3 x 47 mm
- board text added: "AIF_RC遠隔操縦基板 Ver.0.1 設計：kyo0221"
- board text added: "状態表示"
- board text removed: "43x25mm"
- board text removed: "AIF_RC遠隔操縦基板 Ver.0.0 設計：kyo0221"
- board text removed: "ER6"

Commit message: fix: 隠れているシルク印字を修正
Other:
- board text added: "PWR"
Changed lines of the file:
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@@
 		(tags "capacitor")
 		(property "Reference" "C16"
-			(at 7.525 1.4 90)
+			(at 0 -1.4 90)
 			(layer "F.SilkS")
 			(effects
@@
 		(tags "capacitor")
 		(property "Reference" "C12"
-			(at 2.204819 0 90)
+			(at 0 -1.2 180)
 			(layer "F.SilkS")
 			(effects
@@
 		(tags "resistor")
 		(property "Reference" "R7"
-			(at -0.047619 -1.454819 90)
+			(at -2.025 0 180)
 			(layer "F.SilkS")
 			(effects
@@
 		)
 	)
+	(gr_text "PWR"
+		(at 159.8 56.4 90)
+		(layer "Dwgs.User")
+		(effects
+			(font
+				(size 1 1)
+				(thickness 0.15)
+			)
+			(justify left bottom)
+		)
+	)

Commit message: fix: 添削内容を踏まえて修正
Parts:
- moved R1 18.8 mm to (196.0, 90.6), turned to -90 degrees
- moved C6 16.1 mm to (178.7, 72.3), turned to 0 degrees
- moved J3 9.36 mm to (182.0, 94.0)
- moved G*** 8.02 mm to (158.1, 88.7)
- moved H4 7.59 mm to (197.0, 97.0)
- moved H3 7.47 mm to (153.0, 97.0)
- moved SW1 5.12 mm to (181.2, 87.7)
- moved JP1 3.95 mm to (196.0, 87.0), turned to 180 degrees
- moved H2 2.82 mm to (197.0, 53.0)
- moved H1 2.50 mm to (153.0, 53.0)
- moved C4 2.48 mm to (172.2, 61.5), turned to -90 degrees
- moved J4 2.06 mm to (196.0, 79.0), turned to 90 degrees
- moved C20 1.00 mm to (179.6, 61.8)
- moved C1 0.60 mm to (174.0, 61.9)
- moved C2 0.60 mm to (176.0, 61.8)
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Connections:
- U1 pad 17: unconnected-(U1-PA3-Pad17) -> /STM32G474/STATUS_LED
- U1 pad 18: unconnected-(U1-PA4-Pad18) -> /STM32G474/FAIL_LED
- U1 pad 19: unconnected-(U1-PA5-Pad19) -> /STM32G474/MODE_LED
- U1 pad 24: /STM32G474/STATUS_LED -> unconnected-(U1-PB0-Pad24)
- U1 pad 25: /STM32G474/FAIL_LED -> unconnected-(U1-PB1-Pad25)
- U1 pad 26: /STM32G474/MODE_LED -> unconnected-(U1-PB2-Pad26)
Routing:
- net /CAN_Transeiver/CAN_RX: track 60.1 -> 30.0 mm, vias 0 -> 2
- net +3.3V: track 137.2 -> 112.5 mm, vias 6 -> 7
- net /CAN_Transeiver/CAN_TX: track 51.2 -> 34.9 mm, vias 0 -> 2
- net /CAN_Transeiver/GND_CAN: track 15.5 -> 0.00 mm, vias 2 -> 40
- net /CAN_Transeiver/CAN_L: track 13.8 -> 28.3 mm, vias 0 -> 1
- net Net-(JP1-A): track 12.2 -> 2.81 mm
- net +5V: track 0.00 -> 3.16 mm
- net /STM32G474/SWDIO: track 9.67 -> 12.5 mm
- net /STM32G474/FAIL_LED: track 10.2 -> 7.33 mm, vias 2 -> 0
- net /STM32G474/STATUS_LED: track 9.22 -> 6.55 mm
- net /STM32G474/SWCLK: track 11.2 -> 13.5 mm
- net /STM32G474/MODE_LED: track 16.9 -> 19.0 mm
- net GND: track 18.4 -> 16.4 mm, vias 76 -> 146
- net /USART_TX: track 29.4 -> 27.4 mm, vias 6 -> 1
- net /STM32G474/SWO: track 14.7 -> 16.5 mm
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- added copper zone on B.Cu, net /CAN_Transeiver/GND_CAN
Other:
- board size 48.3 x 47 mm -> 50 x 50 mm
- board text added: "AIF_RC遠隔操縦基板 Ver.0.2 設計：kyo0221"
- board text added: "RST"
- board text added: "手動"
- board text removed: "AIF_RC遠隔操縦基板 Ver.0.1 設計：kyo0221"
- board text removed: "モード"
- board text removed: "状態表示"
